File: Projekt/Thermometer/Thermometer.kicad_pcb (KiCad board)
At the start: 4 copper layers, 89 x 81 mm, 5 parts, among them J1 Conn_01x09_Socket, U1 RC1602A, U2 DHT11_Module

Commit message: no progress
Parts:
- renumbered J1 to ARDUINO, U2 to DHT11, U1 to LCD, RV1 to POTENTIOMETER
Other:
- board text added: "220"
- board text added: "THERMOMETER"
Changed lines of the file:
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@@
 		(descr "LCD 16x2 http://www.wincomlcd.com/pdf/WC1602A-SFYLYHTC06.pdf")
 		(tags "LCD 16x2 Alphanumeric 16pin")
-		(property "Reference" "U1"
+		(property "Reference" "LCD"
 			(at -5.82 -3.81 0)
 			(layer "F.SilkS")
@@
 		(descr "Through hole straight socket strip, 1x09, 2.54mm pitch, single row (from Kicad 4.0.7), script generated")
 		(tags "Through hole socket strip THT 1x09 2.54mm single row")
-		(property "Reference" "J1"
+		(property "Reference" "ARDUINO"
 			(at 0 -2.77 90)
 			(layer "F.SilkS")
@@
 		(descr "Potentiometer, vertical, ACP CA9-V10, http://www.acptechnologies.com/wp-content/uploads/2017/05/02-ACP-CA9-CE9.pdf")
 		(tags "Potentiometer vertical ACP CA9-V10")
-		(property "Reference" "RV1"
+		(property "Reference" "POTENTIOMETER"
 			(at 5 -8.65 90)
 			(layer "F.SilkS")
@@
 		(descr "Through hole straight socket strip, 1x03, 2.00mm pitch, single row (from Kicad 4.0.7), script generated")
 		(tags "Through hole socket strip THT 1x03 2.00mm single row")
-		(property "Reference" "U2"
+		(property "Reference" "DHT11"
 			(at 0 -2.5 90)
 			(layer "F.SilkS")
@@
 	)
 	(gr_text "D8"
-		(at 64.4 82.1 90)
+		(at 64.4 83.8 90)
 		(layer "F.Cu")
 		(effects
@@
 		)
 	)
+	(gr_text "220"
+		(at 94.95 89.8 90)
+		(layer "F.Cu")
+		(effects
+			(font
+				(size 1.5 1.5)
+				(thickness 0.3)
+				(bold yes)
+			)
+			(justify left bottom)
+		)
+	)
+	(gr_text "THERMOMETER"
+		(at 46.1 58.9 0)
+		(layer "F.Cu")
+		(effects
+			(font
+				(size 1.8 1.8)
+				(thickness 0.3)
+				(bold yes)
+			)
+			(justify left bottom)
+		)
+	)
 	(segment
 		(start 93.98 83.82)
@@
 		(layer "F.Cu")
 		(net "Net-(U1-VO)")
+	)
+	(segment
+		(start 66 77.04)
+		(end 66.04 77)
+		(width 0.2)
+		(layer "F.Cu")
+		(net "Net-(J1-Pin_8)")
+	)
+	(segment
+		(start 66.04 94.04)
+		(end 66.04 99.06)
+		(width 0.2)
+		(layer "F.Cu")
+		(net "Net-(J1-Pin_8)")
+	)
+	(segment
+		(start 66 94)
+		(end 66.04 94.04)
+		(width 0.2)
+		(layer "F.Cu")
+		(net "Net-(J1-Pin_8)")
+	)
+	(segment
+		(start 66 78.9)
+		(end 66 77.04)
+		(width 0.2)
+		(layer "F.Cu")
+		(net "Net-(J1-Pin_8)")
+	)
+	(via
+		(at 66 78.9)
+		(size 0.7)
+		(drill 0.3)
+		(layers "F.Cu" "B.Cu")
+		(net "Net-(J1-Pin_8)")
+	)
+	(via
+		(at 66 94)
+		(size 0.7)
+		(drill 0.3)
+		(layers "F.Cu" "B.Cu")
+		(net "Net-(J1-Pin_8)")
+	)
+	(segment
+		(start 66 94)
+		(end 66 78.9)
+		(width 0.2)
+		(layer "B.Cu")
+		(net "Net-(J1-Pin_8)")
 	)
 	(segment
@@
 	)
 	(segment
+		(start 71.12 77.07)
+		(end 73.7 79.65)
+		(width 0.2)
+		(layer "F.Cu")
+		(net "Net-(J1-Pin_6)")
+	)
+	(segment
+		(start 71.12 77)
+		(end 71.12 77.07)
+		(width 0.2)
+		(layer "F.Cu")
+		(net "Net-(J1-Pin_6)")
+	)
+	(segment
+		(start 83.82 99.06)
+		(end 83.82 89.7)
+		(width 0.2)
+		(layer "F.Cu")
+		(net "Net-(J1-Pin_6)")
+	)
+	(via
+		(at 83.82 89.7)
+		(size 0.7)
+		(drill 0.3)
+		(layers "F.Cu" "B.Cu")
+		(net "Net-(J1-Pin_6)")
+	)
+	(via
+		(at 73.7 79.65)
+		(size 0.7)
+		(drill 0.3)
+		(layers "F.Cu" "B.Cu")
+		(net "Net-(J1-Pin_6)")
+	)
+	(segment
+		(start 73.7 79.65)
+		(end 83.75 89.7)
+		(width 0.2)
+		(layer "B.Cu")
+		(net "Net-(J1-Pin_6)")
+	)
+	(segment
+		(start 83.75 89.7)
+		(end 83.82 89.7)
+		(width 0.2)
+		(layer "B.Cu")
+		(net "Net-(J1-Pin_6)")
+	)
+	(segment
+		(start 73.66 77)
+		(end 76.2 79.54)
+		(width 0.2)
+		(layer "F.Cu")
+		(net "Net-(J1-Pin_5)")
+	)
+	(segment
+		(start 86.36 89.7)
+		(end 86.36 99.06)
+		(width 0.2)
+		(layer "F.Cu")
+		(net "Net-(J1-Pin_5)")
+	)
+	(segment
+		(start 76.2 79.54)
+		(end 76.2 79.55)
+		(width 0.2)
+		(layer "F.Cu")
+		(net "Net-(J1-Pin_5)")
+	)
+	(via
+		(at 86.36 89.7)
+		(size 0.7)
+		(drill 0.3)
+		(layers "F.Cu" "B.Cu")
+		(net "Net-(J1-Pin_5)")
+	)
+	(via
+		(at 76.2 79.55)
+		(size 0.7)
+		(drill 0.3)
+		(layers "F.Cu" "B.Cu")
+		(net "Net-(J1-Pin_5)")
+	)
+	(segment
+		(start 76.2 79.55)
+		(end 86.35 89.7)
+		(width 0.2)
+		(layer "B.Cu")
+		(net "Net-(J1-Pin_5)")
+	)
+	(segment
+		(start 86.35 89.7)
+		(end 86.36 89.7)
+		(width 0.2)
+		(layer "B.Cu")
+		(net "Net-(J1-Pin_5)")
+	)
+	(segment
 		(start 76.2 77)
 		(end 78.65 79.45)
@@
 		(net "Net-(J1-Pin_9)")
 	)
-	(segment
-		(start 66 77.04)
-		(end 66.04 77)
-		(width 0.2)
-		(layer "F.Cu")
-		(net "Net-(J1-Pin_8)")
-	)
-	(segment
-		(start 66.04 94.04)
-		(end 66.04 99.06)
-		(width 0.2)
-		(layer "F.Cu")
-		(net "Net-(J1-Pin_8)")
-	)
-	(segment
-		(start 66 94)
-		(end 66.04 94.04)
-		(width 0.2)
-		(layer "F.Cu")
-		(net "Net-(J1-Pin_8)")
-	)
-	(segment
-		(start 66 78.9)
-		(end 66 77.04)
-		(width 0.2)
-		(layer "F.Cu")
-		(net "Net-(J1-Pin_8)")
-	)
-	(via
-		(at 66 78.9)
-		(size 0.7)
-		(drill 0.3)
-		(layers "F.Cu" "B.Cu")
-		(net "Net-(J1-Pin_8)")
-	)
-	(via
-		(at 66 94)
-		(size 0.7)
-		(drill 0.3)
-		(layers "F.Cu" "B.Cu")
-		(net "Net-(J1-Pin_8)")
-	)
-	(segment
-		(start 66 94)
-		(end 66 78.9)
-		(width 0.2)
-		(layer "B.Cu")
-		(net "Net-(J1-Pin_8)")
-	)
-	(segment
-		(start 71.12 77.07)
-		(end 73.7 79.65)
-		(width 0.2)
-		(layer "F.Cu")
-		(net "Net-(J1-Pin_6)")
-	)
-	(segment
-		(start 71.12 77)
-		(end 71.12 77.07)
-		(width 0.2)
-		(layer "F.Cu")
-		(net "Net-(J1-Pin_6)")
-	)
-	(segment
-		(start 83.82 99.06)
-		(end 83.82 89.7)
-		(width 0.2)
-		(layer "F.Cu")
-		(net "Net-(J1-Pin_6)")
-	)
-	(via
-		(at 83.82 89.7)
-		(size 0.7)
-		(drill 0.3)
-		(layers "F.Cu" "B.Cu")
-		(net "Net-(J1-Pin_6)")
-	)
-	(via
-		(at 73.7 79.65)
-		(size 0.7)
-		(drill 0.3)
-		(layers "F.Cu" "B.Cu")
-		(net "Net-(J1-Pin_6)")
-	)
-	(segment
-		(start 73.7 79.65)
-		(end 83.75 89.7)
-		(width 0.2)
-		(layer "B.Cu")
-		(net "Net-(J1-Pin_6)")
-	)
-	(segment
-		(start 83.75 89.7)
-		(end 83.82 89.7)
-		(width 0.2)
-		(layer "B.Cu")
-		(net "Net-(J1-Pin_6)")
-	)
-	(segment
-		(start 73.66 77)
-		(end 76.2 79.54)
-		(width 0.2)
-		(layer "F.Cu")
-		(net "Net-(J1-Pin_5)")
-	)
-	(segment
-		(start 86.36 89.7)
-		(end 86.36 99.06)
-		(width 0.2)
-		(layer "F.Cu")
-		(net "Net-(J1-Pin_5)")
-	)
-	(segment
-		(start 76.2 79.54)
-		(end 76.2 79.55)
-		(width 0.2)
-		(layer "F.Cu")
-		(net "Net-(J1-Pin_5)")
-	)
-	(via
-		(at 86.36 89.7)
-		(size 0.7)
-		(drill 0.3)
-		(layers "F.Cu" "B.Cu")
-		(net "Net-(J1-Pin_5)")
-	)
-	(via
-		(at 76.2 79.55)
-		(size 0.7)
-		(drill 0.3)
-		(layers "F.Cu" "B.Cu")
-		(net "Net-(J1-Pin_5)")
-	)
-	(segment
-		(start 76.2 79.55)
-		(end 86.35 89.7)
-		(width 0.2)
-		(layer "B.Cu")
-		(net "Net-(J1-Pin_5)")
-	)
-	(segment
-		(start 86.35 89.7)
-		(end 86.36 89.7)
-		(width 0.2)
-		(layer "B.Cu")
-		(net "Net-(J1-Pin_5)")
-	)
 	(zone
